File: hardware/sweet sixteen v24_3.sch (EAGLE design)
At the start: 204 parts, among them IC1 LM4040C25, IC2 LM4040c50, IC3 LM1117-5, IC4 UA78M08DCY, J1 PJ301_THONKICONN6, J10 PJ301_THONKICONN6, J11 PJ301_THONKICONN6, J12 PJ301_THONKICONN6, J13 PJ301_THONKICONN6, J14 PJ301_THONKICONN6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

Commit message: Add files via upload
Other:
- note added: "Maangu Díaz 2019"
- note added: "tesseract.modular@gmail.com"
- note removed: "Olivier Gillet"
- note removed: "ol.gillet@gmail.com"
- moved on the sheet: C17, C18, C5, C8
